Commit message: motors

File: body.urdf (robot description, URDF)
Before this commit: robot robot, 3 links, 2 joints
Joints:
- removed joint Torse_Frontleg
- added joint Torso_Frontleg: type revolute, parent Torso, child Frontleg, origin xyz=1.5 0 1 rpy=0 0 0, axis 0 1 0, limit lower=-3.14159 upper=3.14159 effort=0.0 velocity=0.0

Commit message: finishing

File: body.urdf (robot description, URDF)
Before this commit: robot robot, 3 links, 2 joints
Links:
- removed link Backleg
- removed link Frontleg
- added link BackLeg, mass 1; collision box size=0.2 1 0.2; visual box size=0.2 1 0.2
- added link BackLower, mass 1; collision box size=0.2 0.2 1; visual box size=0.2 0.2 1
- added link FrontLeg, mass 1; collision box size=0.2 1 0.2; visual box size=0.2 1 0.2
- added link FrontLower, mass 1; collision box size=0.2 0.2 1; visual box size=0.2 0.2 1
- added link LeftLeg, mass 1; collision box size=1 0.2 0.2; visual box size=1 0.2 0.2
- added link LeftLower, mass 1; collision box size=0.2 0.2 1; visual box size=0.2 0.2 1
- added link RightLeg, mass 1; collision box size=1 0.2 0.2; visual box size=1 0.2 0.2
- added link RightLower, mass 1; collision box size=0.2 0.2 1; visual box size=0.2 0.2 1
Joints:
- removed joint Torso_Backleg
- removed joint Torso_Frontleg
- added joint BackLeg_BackLower: type revolute, parent BackLeg, child BackLower, origin xyz=0 -1 0 rpy=0 0 0, axis 1 0 1, limit lower=-3.14159 upper=3.14159 effort=0.0 velocity=0.0
- added joint FrontLeg_FrontLower: type revolute, parent FrontLeg, child FrontLower, origin xyz=0 1 0 rpy=0 0 0, axis 1 0 1, limit lower=-3.14159 upper=3.14159 effort=0.0 velocity=0.0
- added joint LeftLeg_LeftLower: type revolute, parent LeftLeg, child LeftLower, origin xyz=-1 0 0 rpy=0 0 0, axis 0 1 1, limit lower=-3.14159 upper=3.14159 effort=0.0 velocity=0.0
- added joint RightLeg_RightLower: type revolute, parent RightLeg, child RightLower, origin xyz=1 0 0 rpy=0 0 0, axis 0 1 1, limit lower=-3.14159 upper=3.14159 effort=0.0 velocity=0.0
- added joint Torso_BackLeg: type revolute, parent Torso, child BackLeg, origin xyz=0 -0.5 1 rpy=0 0 0, axis 1 0 1, limit lower=-3.14159 upper=3.14159 effort=0.0 velocity=0.0
- added joint Torso_FrontLeg: type revolute, parent Torso, child FrontLeg, origin xyz=0 0.5 1 rpy=0 0 0, axis 1 0 1, limit lower=-3.14159 upper=3.14159 effort=0.0 velocity=0.0
- added joint Torso_LeftLeg: type revolute, parent Torso, child LeftLeg, origin xyz=-0.5 0 1 rpy=0 0 0, axis 0 1 1, limit lower=-3.14159 upper=3.14159 effort=0.0 velocity=0.0
- added joint Torso_RightLeg: type revolute, parent Torso, child RightLeg, origin xyz=0.5 0 1 rpy=0 0 0, axis 0 1 1, limit lower=-3.14159 upper=3.14159 effort=0.0 velocity=0.0
