Commit message: spinny ball

File: body151.urdf (robot description, URDF)
Before this commit: robot robot, 9 links, 8 joints
Joints:
- joint Torso_BackLeg: origin xyz=0 -0.5 1 rpy=0 0 0 -> xyz=0 4.5 1 rpy=0 0 0
- joint Torso_FrontLeg: origin xyz=0 0.5 1 rpy=0 0 0 -> xyz=0 5.5 1 rpy=0 0 0
- joint Torso_LeftLeg: origin xyz=-0.5 0 1 rpy=0 0 0 -> xyz=-0.5 5 1 rpy=0 0 0
- joint Torso_RightLeg: origin xyz=0.5 0 1 rpy=0 0 0 -> xyz=0.5 5 1 rpy=0 0 0
