Commit message: code dump

File: body0.urdf (robot description, URDF)
Before this commit: robot robot, 9 links, 8 joints
Links:
- link BackLeg: geometry collision box size=0 0 0; visual box size=0 0 0
- link BackLower: geometry collision box size=0 0 0; visual box size=0 0 0
- link FrontLeg: geometry collision box size=0 0 0; visual box size=0 0 0
- link FrontLower: geometry collision box size=0 0 0; visual box size=0 0 0
- link LeftLeg: geometry collision box size=0 0 0; visual box size=0 0 0
- link LeftLower: geometry collision box size=0 0 0; visual box size=0 0 0
- link RightLeg: geometry collision box size=0 0 0; visual box size=0 0 0
- link RightLower: geometry collision box size=0 0 0; visual box size=0 0 0
- link Torso: geometry collision sphere radius=1 1 1; visual sphere radius=1 1 1
