Commit message: voxel cilia model

File: body0.urdf (robot description, URDF)
Before this commit: robot robot, 9 links, 8 joints
Links:
- removed link BackLeg
- removed link BackLower
- removed link FrontLeg
- removed link FrontLower
- removed link LeftLeg
- removed link LeftLower
- removed link RightLeg
- removed link RightLower
- removed link Torso
- added link 123, mass 1; collision box size=0.1 0.1 0.1; visual box size=0.1 0.1 0.1
- added link 124, mass 1; collision box size=0.1 0.1 0.1; visual box size=0.1 0.1 0.1
- added link 125, mass 1; collision box size=0.1 0.1 0.1; visual box size=0.1 0.1 0.1
- added link 132, mass 1; collision box size=0.1 0.1 0.1; visual box size=0.1 0.1 0.1
- added link 133, mass 1; collision box size=0.1 0.1 0.1; visual box size=0.1 0.1 0.1
- added link 134, mass 1; collision box size=0.1 0.1 0.1; visual box size=0.1 0.1 0.1
- added link 135, mass 1; collision box size=0.1 0.1 0.1; visual box size=0.1 0.1 0.1
- added link 136, mass 1; collision box size=0.1 0.1 0.1; visual box size=0.1 0.1 0.1
- added link 142, mass 1; collision box size=0.1 0.1 0.1; visual box size=0.1 0.1 0.1
- added link 143, mass 1; collision box size=0.1 0.1 0.1; visual box size=0.1 0.1 0.1
- added link 144, mass 1; collision box size=0.1 0.1 0.1; visual box size=0.1 0.1 0.1
- added link 145, mass 1; collision box size=0.1 0.1 0.1; visual box size=0.1 0.1 0.1
- added link 146, mass 1; collision box size=0.1 0.1 0.1; visual box size=0.1 0.1 0.1
- added link 152, mass 1; collision box size=0.1 0.1 0.1; visual box size=0.1 0.1 0.1
- added link 153, mass 1; collision box size=0.1 0.1 0.1; visual box size=0.1 0.1 0.1
- added link 154, mass 1; collision box size=0.1 0.1 0.1; visual box size=0.1 0.1 0.1
- added link 155, mass 1; collision box size=0.1 0.1 0.1; visual box size=0.1 0.1 0.1
- added link 156, mass 1; collision box size=0.1 0.1 0.1; visual box size=0.1 0.1 0.1
- added link 163, mass 1; collision box size=0.1 0.1 0.1; visual box size=0.1 0.1 0.1
- added link 164, mass 1; collision box size=0.1 0.1 0.1; visual box size=0.1 0.1 0.1
- added link 165, mass 1; collision box size=0.1 0.1 0.1; visual box size=0.1 0.1 0.1
- added link 213, mass 1; collision box size=0.1 0.1 0.1; visual box size=0.1 0.1 0.1
- added link 214, mass 1; collision box size=0.1 0.1 0.1; visual box size=0.1 0.1 0.1
- added link 215, mass 1; collision box size=0.1 0.1 0.1; visual box size=0.1 0.1 0.1
- added link 222, mass 1; collision box size=0.1 0.1 0.1; visual box size=0.1 0.1 0.1
- added link 226, mass 1; collision box size=0.1 0.1 0.1; visual box size=0.1 0.1 0.1
- added link 231, mass 1; collision box size=0.1 0.1 0.1; visual box size=0.1 0.1 0.1
- added link 241, mass 1; collision box size=0.1 0.1 0.1; visual box size=0.1 0.1 0.1
- added link 251, mass 1; collision box size=0.1 0.1 0.1; visual box size=0.1 0.1 0.1
- added link 262, mass 1; collision box size=0.1 0.1 0.1; visual box size=0.1 0.1 0.1
- added link 266, mass 1; collision box size=0.1 0.1 0.1; visual box size=0.1 0.1 0.1
- added link 273, mass 1; collision box size=0.1 0.1 0.1; visual box size=0.1 0.1 0.1
- added link 274, mass 1; collision box size=0.1 0.1 0.1; visual box size=0.1 0.1 0.1
- added link 275, mass 1; collision box size=0.1 0.1 0.1; visual box size=0.1 0.1 0.1
- added link 312, mass 1; collision box size=0.1 0.1 0.1; visual box size=0.1 0.1 0.1
- added link 313, mass 1; collision box size=0.1 0.1 0.1; visual box size=0.1 0.1 0.1
- added link 314, mass 1; collision box size=0.1 0.1 0.1; visual box size=0.1 0.1 0.1
- added link 315, mass 1; collision box size=0.1 0.1 0.1; visual box size=0.1 0.1 0.1
- added link 316, mass 1; collision box size=0.1 0.1 0.1; visual box size=0.1 0.1 0.1
- added link 321, mass 1; collision box size=0.1 0.1 0.1; visual box size=0.1 0.1 0.1
- added link 331, mass 1; collision box size=0.1 0.1 0.1; visual box size=0.1 0.1 0.1
- added link 341, mass 1; collision box size=0.1 0.1 0.1; visual box size=0.1 0.1 0.1
- added link 351, mass 1; collision box size=0.1 0.1 0.1; visual box size=0.1 0.1 0.1
- added link 361, mass 1; collision box size=0.1 0.1 0.1; visual box size=0.1 0.1 0.1
- added link 372, mass 1; collision box size=0.1 0.1 0.1; visual box size=0.1 0.1 0.1
- added link 373, mass 1; collision box size=0.1 0.1 0.1; visual box size=0.1 0.1 0.1
- added link 374, mass 1; collision box size=0.1 0.1 0.1; visual box size=0.1 0.1 0.1
- added link 375, mass 1; collision box size=0.1 0.1 0.1; visual box size=0.1 0.1 0.1
- added link 376, mass 1; collision box size=0.1 0.1 0.1; visual box size=0.1 0.1 0.1
- added link 412, mass 1; collision box size=0.1 0.1 0.1; visual box size=0.1 0.1 0.1
- added link 413, mass 1; collision box size=0.1 0.1 0.1; visual box size=0.1 0.1 0.1
- added link 414, mass 1; collision box size=0.1 0.1 0.1; visual box size=0.1 0.1 0.1
- added link 415, mass 1; collision box size=0.1 0.1 0.1; visual box size=0.1 0.1 0.1
- added link 416, mass 1; collision box size=0.1 0.1 0.1; visual box size=0.1 0.1 0.1
- added link 421, mass 1; collision box size=0.1 0.1 0.1; visual box size=0.1 0.1 0.1
- added link 431, mass 1; collision box size=0.1 0.1 0.1; visual box size=0.1 0.1 0.1
- added link 440, mass 1; collision box size=0 0 0; visual box size=0 0 0
- added link 441, mass 1; collision box size=0.1 0.1 0.1; visual box size=0.1 0.1 0.1
- added link 451, mass 1; collision box size=0.1 0.1 0.1; visual box size=0.1 0.1 0.1
- added link 461, mass 1; collision box size=0.1 0.1 0.1; visual box size=0.1 0.1 0.1
- added link 472, mass 1; collision box size=0.1 0.1 0.1; visual box size=0.1 0.1 0.1
- added link 473, mass 1; collision box size=0.1 0.1 0.1; visual box size=0.1 0.1 0.1
- added link 474, mass 1; collision box size=0.1 0.1 0.1; visual box size=0.1 0.1 0.1
- added link 475, mass 1; collision box size=0.1 0.1 0.1; visual box size=0.1 0.1 0.1
- added link 476, mass 1; collision box size=0.1 0.1 0.1; visual box size=0.1 0.1 0.1
- added link 512, mass 1; collision box size=0.1 0.1 0.1; visual box size=0.1 0.1 0.1
- added link 513, mass 1; collision box size=0.1 0.1 0.1; visual box size=0.1 0.1 0.1
- added link 514, mass 1; collision box size=0.1 0.1 0.1; visual box size=0.1 0.1 0.1
- added link 515, mass 1; collision box size=0.1 0.1 0.1; visual box size=0.1 0.1 0.1
- added link 516, mass 1; collision box size=0.1 0.1 0.1; visual box size=0.1 0.1 0.1
- added link 521, mass 1; collision box size=0.1 0.1 0.1; visual box size=0.1 0.1 0.1
- added link 531, mass 1; collision box size=0.1 0.1 0.1; visual box size=0.1 0.1 0.1
- added link 541, mass 1; collision box size=0.1 0.1 0.1; visual box size=0.1 0.1 0.1
- added link 551, mass 1; collision box size=0.1 0.1 0.1; visual box size=0.1 0.1 0.1
- added link 561, mass 1; collision box size=0.1 0.1 0.1; visual box size=0.1 0.1 0.1
- added link 572, mass 1; collision box size=0.1 0.1 0.1; visual box size=0.1 0.1 0.1
- added link 573, mass 1; collision box size=0.1 0.1 0.1; visual box size=0.1 0.1 0.1
- added link 574, mass 1; collision box size=0.1 0.1 0.1; visual box size=0.1 0.1 0.1
- added link 575, mass 1; collision box size=0.1 0.1 0.1; visual box size=0.1 0.1 0.1
- added link 576, mass 1; collision box size=0.1 0.1 0.1; visual box size=0.1 0.1 0.1
- added link 613, mass 1; collision box size=0.1 0.1 0.1; visual box size=0.1 0.1 0.1
- added link 614, mass 1; collision box size=0.1 0.1 0.1; visual box size=0.1 0.1 0.1
- added link 615, mass 1; collision box size=0.1 0.1 0.1; visual box size=0.1 0.1 0.1
- added link 622, mass 1; collision box size=0.1 0.1 0.1; visual box size=0.1 0.1 0.1
- added link 626, mass 1; collision box size=0.1 0.1 0.1; visual box size=0.1 0.1 0.1
- added link 631, mass 1; collision box size=0.1 0.1 0.1; visual box size=0.1 0.1 0.1
- added link 641, mass 1; collision box size=0.1 0.1 0.1; visual box size=0.1 0.1 0.1
- added link 651, mass 1; collision box size=0.1 0.1 0.1; visual box size=0.1 0.1 0.1
- added link 662, mass 1; collision box size=0.1 0.1 0.1; visual box size=0.1 0.1 0.1
- added link 666, mass 1; collision box size=0.1 0.1 0.1; visual box size=0.1 0.1 0.1
- added link 673, mass 1; collision box size=0.1 0.1 0.1; visual box size=0.1 0.1 0.1
- added link 674, mass 1; collision box size=0.1 0.1 0.1; visual box size=0.1 0.1 0.1
- added link 675, mass 1; collision box size=0.1 0.1 0.1; visual box size=0.1 0.1 0.1
- added link 723, mass 1; collision box size=0.1 0.1 0.1; visual box size=0.1 0.1 0.1
- added link 724, mass 1; collision box size=0.1 0.1 0.1; visual box size=0.1 0.1 0.1
- added link 725, mass 1; collision box size=0.1 0.1 0.1; visual box size=0.1 0.1 0.1
- added link 732, mass 1; collision box size=0.1 0.1 0.1; visual box size=0.1 0.1 0.1
- added link 733, mass 1; collision box size=0.1 0.1 0.1; visual box size=0.1 0.1 0.1
- added link 734, mass 1; collision box size=0.1 0.1 0.1; visual box size=0.1 0.1 0.1
- added link 735, mass 1; collision box size=0.1 0.1 0.1; visual box size=0.1 0.1 0.1
- added link 736, mass 1; collision box size=0.1 0.1 0.1; visual box size=0.1 0.1 0.1
- added link 742, mass 1; collision box size=0.1 0.1 0.1; visual box size=0.1 0.1 0.1
- added link 743, mass 1; collision box size=0.1 0.1 0.1; visual box size=0.1 0.1 0.1
- added link 744, mass 1; collision box size=0.1 0.1 0.1; visual box size=0.1 0.1 0.1
- added link 745, mass 1; collision box size=0.1 0.1 0.1; visual box size=0.1 0.1 0.1
- added link 746, mass 1; collision box size=0.1 0.1 0.1; visual box size=0.1 0.1 0.1
- added link 752, mass 1; collision box size=0.1 0.1 0.1; visual box size=0.1 0.1 0.1
- added link 753, mass 1; collision box size=0.1 0.1 0.1; visual box size=0.1 0.1 0.1
- added link 754, mass 1; collision box size=0.1 0.1 0.1; visual box size=0.1 0.1 0.1
- added link 755, mass 1; collision box size=0.1 0.1 0.1; visual box size=0.1 0.1 0.1
- added link 756, mass 1; collision box size=0.1 0.1 0.1; visual box size=0.1 0.1 0.1
- added link 763, mass 1; collision box size=0.1 0.1 0.1; visual box size=0.1 0.1 0.1
- added link 764, mass 1; collision box size=0.1 0.1 0.1; visual box size=0.1 0.1 0.1
- added link 765, mass 1; collision box size=0.1 0.1 0.1; visual box size=0.1 0.1 0.1
Joints:
- removed joint BackLeg_BackLower
- removed joint FrontLeg_FrontLower
- removed joint LeftLeg_LeftLower
- removed joint RightLeg_RightLower
- removed joint Torso_BackLeg
- removed joint Torso_FrontLeg
- removed joint Torso_LeftLeg
- removed joint Torso_RightLeg
- added joint 440_123: type fixed, parent 440, child 123, origin xyz=0   0 rpy=0 0 0, axis 0 0 1, limit lower=-3.14159 upper=3.14159 effort=0.0 velocity=0.0
- added joint 440_124: type fixed, parent 440, child 124, origin xyz=0   0 rpy=0 0 0, axis 0 0 1, limit lower=-3.14159 upper=3.14159 effort=0.0 velocity=0.0
- added joint 440_125: type fixed, parent 440, child 125, origin xyz=0   0 rpy=0 0 0, axis 0 0 1, limit lower=-3.14159 upper=3.14159 effort=0.0 velocity=0.0
- added joint 440_132: type fixed, parent 440, child 132, origin xyz=0   0 rpy=0 0 0, axis 0 0 1, limit lower=-3.14159 upper=3.14159 effort=0.0 velocity=0.0
- added joint 440_133: type fixed, parent 440, child 133, origin xyz=0   0 rpy=0 0 0, axis 0 0 1, limit lower=-3.14159 upper=3.14159 effort=0.0 velocity=0.0
- added joint 440_134: type fixed, parent 440, child 134, origin xyz=0   0 rpy=0 0 0, axis 0 0 1, limit lower=-3.14159 upper=3.14159 effort=0.0 velocity=0.0
- added joint 440_135: type fixed, parent 440, child 135, origin xyz=0   0 rpy=0 0 0, axis 0 0 1, limit lower=-3.14159 upper=3.14159 effort=0.0 velocity=0.0
- added joint 440_136: type fixed, parent 440, child 136, origin xyz=0   0 rpy=0 0 0, axis 0 0 1, limit lower=-3.14159 upper=3.14159 effort=0.0 velocity=0.0
- added joint 440_142: type fixed, parent 440, child 142, origin xyz=0   0 rpy=0 0 0, axis 0 0 1, limit lower=-3.14159 upper=3.14159 effort=0.0 velocity=0.0
- added joint 440_143: type fixed, parent 440, child 143, origin xyz=0   0 rpy=0 0 0, axis 0 0 1, limit lower=-3.14159 upper=3.14159 effort=0.0 velocity=0.0
- added joint 440_144: type fixed, parent 440, child 144, origin xyz=0   0 rpy=0 0 0, axis 0 0 1, limit lower=-3.14159 upper=3.14159 effort=0.0 velocity=0.0
- added joint 440_145: type fixed, parent 440, child 145, origin xyz=0   0 rpy=0 0 0, axis 0 0 1, limit lower=-3.14159 upper=3.14159 effort=0.0 velocity=0.0
- added joint 440_146: type fixed, parent 440, child 146, origin xyz=0   0 rpy=0 0 0, axis 0 0 1, limit lower=-3.14159 upper=3.14159 effort=0.0 velocity=0.0
- added joint 440_152: type fixed, parent 440, child 152, origin xyz=0   0 rpy=0 0 0, axis 0 0 1, limit lower=-3.14159 upper=3.14159 effort=0.0 velocity=0.0
- added joint 440_153: type fixed, parent 440, child 153, origin xyz=0   0 rpy=0 0 0, axis 0 0 1, limit lower=-3.14159 upper=3.14159 effort=0.0 velocity=0.0
- added joint 440_154: type fixed, parent 440, child 154, origin xyz=0   0 rpy=0 0 0, axis 0 0 1, limit lower=-3.14159 upper=3.14159 effort=0.0 velocity=0.0
- added joint 440_155: type fixed, parent 440, child 155, origin xyz=0   0 rpy=0 0 0, axis 0 0 1, limit lower=-3.14159 upper=3.14159 effort=0.0 velocity=0.0
- added joint 440_156: type fixed, parent 440, child 156, origin xyz=0   0 rpy=0 0 0, axis 0 0 1, limit lower=-3.14159 upper=3.14159 effort=0.0 velocity=0.0
- added joint 440_163: type fixed, parent 440, child 163, origin xyz=0   0 rpy=0 0 0, axis 0 0 1, limit lower=-3.14159 upper=3.14159 effort=0.0 velocity=0.0
- added joint 440_164: type fixed, parent 440, child 164, origin xyz=0   0 rpy=0 0 0, axis 0 0 1, limit lower=-3.14159 upper=3.14159 effort=0.0 velocity=0.0
- added joint 440_165: type fixed, parent 440, child 165, origin xyz=0   0 rpy=0 0 0, axis 0 0 1, limit lower=-3.14159 upper=3.14159 effort=0.0 velocity=0.0
- added joint 440_213: type fixed, parent 440, child 213, origin xyz=0   0 rpy=0 0 0, axis 0 0 1, limit lower=-3.14159 upper=3.14159 effort=0.0 velocity=0.0
- added joint 440_214: type fixed, parent 440, child 214, origin xyz=0   0 rpy=0 0 0, axis 0 0 1, limit lower=-3.14159 upper=3.14159 effort=0.0 velocity=0.0
- added joint 440_215: type fixed, parent 440, child 215, origin xyz=0   0 rpy=0 0 0, axis 0 0 1, limit lower=-3.14159 upper=3.14159 effort=0.0 velocity=0.0
- added joint 440_222: type fixed, parent 440, child 222, origin xyz=0   0 rpy=0 0 0, axis 0 0 1, limit lower=-3.14159 upper=3.14159 effort=0.0 velocity=0.0
- added joint 440_226: type fixed, parent 440, child 226, origin xyz=0   0 rpy=0 0 0, axis 0 0 1, limit lower=-3.14159 upper=3.14159 effort=0.0 velocity=0.0
- added joint 440_231: type fixed, parent 440, child 231, origin xyz=0   0 rpy=0 0 0, axis 0 0 1, limit lower=-3.14159 upper=3.14159 effort=0.0 velocity=0.0
- added joint 440_241: type fixed, parent 440, child 241, origin xyz=0   0 rpy=0 0 0, axis 0 0 1, limit lower=-3.14159 upper=3.14159 effort=0.0 velocity=0.0
- added joint 440_251: type fixed, parent 440, child 251, origin xyz=0   0 rpy=0 0 0, axis 0 0 1, limit lower=-3.14159 upper=3.14159 effort=0.0 velocity=0.0
- added joint 440_262: type fixed, parent 440, child 262, origin xyz=0   0 rpy=0 0 0, axis 0 0 1, limit lower=-3.14159 upper=3.14159 effort=0.0 velocity=0.0
- added joint 440_266: type fixed, parent 440, child 266, origin xyz=0   0 rpy=0 0 0, axis 0 0 1, limit lower=-3.14159 upper=3.14159 effort=0.0 velocity=0.0
- added joint 440_273: type fixed, parent 440, child 273, origin xyz=0   0 rpy=0 0 0, axis 0 0 1, limit lower=-3.14159 upper=3.14159 effort=0.0 velocity=0.0
- added joint 440_274: type fixed, parent 440, child 274, origin xyz=0   0 rpy=0 0 0, axis 0 0 1, limit lower=-3.14159 upper=3.14159 effort=0.0 velocity=0.0
- added joint 440_275: type fixed, parent 440, child 275, origin xyz=0   0 rpy=0 0 0, axis 0 0 1, limit lower=-3.14159 upper=3.14159 effort=0.0 velocity=0.0
- added joint 440_312: type fixed, parent 440, child 312, origin xyz=0   0 rpy=0 0 0, axis 0 0 1, limit lower=-3.14159 upper=3.14159 effort=0.0 velocity=0.0
- added joint 440_313: type fixed, parent 440, child 313, origin xyz=0   0 rpy=0 0 0, axis 0 0 1, limit lower=-3.14159 upper=3.14159 effort=0.0 velocity=0.0
- added joint 440_314: type fixed, parent 440, child 314, origin xyz=0   0 rpy=0 0 0, axis 0 0 1, limit lower=-3.14159 upper=3.14159 effort=0.0 velocity=0.0
- added joint 440_315: type fixed, parent 440, child 315, origin xyz=0   0 rpy=0 0 0, axis 0 0 1, limit lower=-3.14159 upper=3.14159 effort=0.0 velocity=0.0
- added joint 440_316: type fixed, parent 440, child 316, origin xyz=0   0 rpy=0 0 0, axis 0 0 1, limit lower=-3.14159 upper=3.14159 effort=0.0 velocity=0.0
- added joint 440_321: type fixed, parent 440, child 321, origin xyz=0   0 rpy=0 0 0, axis 0 0 1, limit lower=-3.14159 upper=3.14159 effort=0.0 velocity=0.0
- added joint 440_331: type fixed, parent 440, child 331, origin xyz=0   0 rpy=0 0 0, axis 0 0 1, limit lower=-3.14159 upper=3.14159 effort=0.0 velocity=0.0
- added joint 440_341: type fixed, parent 440, child 341, origin xyz=0   0 rpy=0 0 0, axis 0 0 1, limit lower=-3.14159 upper=3.14159 effort=0.0 velocity=0.0
- added joint 440_351: type fixed, parent 440, child 351, origin xyz=0   0 rpy=0 0 0, axis 0 0 1, limit lower=-3.14159 upper=3.14159 effort=0.0 velocity=0.0
- added joint 440_361: type fixed, parent 440, child 361, origin xyz=0   0 rpy=0 0 0, axis 0 0 1, limit lower=-3.14159 upper=3.14159 effort=0.0 velocity=0.0
- added joint 440_372: type fixed, parent 440, child 372, origin xyz=0   0 rpy=0 0 0, axis 0 0 1, limit lower=-3.14159 upper=3.14159 effort=0.0 velocity=0.0
- added joint 440_373: type fixed, parent 440, child 373, origin xyz=0   0 rpy=0 0 0, axis 0 0 1, limit lower=-3.14159 upper=3.14159 effort=0.0 velocity=0.0
- added joint 440_374: type fixed, parent 440, child 374, origin xyz=0   0 rpy=0 0 0, axis 0 0 1, limit lower=-3.14159 upper=3.14159 effort=0.0 velocity=0.0
- added joint 440_375: type fixed, parent 440, child 375, origin xyz=0   0 rpy=0 0 0, axis 0 0 1, limit lower=-3.14159 upper=3.14159 effort=0.0 velocity=0.0
- added joint 440_376: type fixed, parent 440, child 376, origin xyz=0   0 rpy=0 0 0, axis 0 0 1, limit lower=-3.14159 upper=3.14159 effort=0.0 velocity=0.0
- added joint 440_412: type fixed, parent 440, child 412, origin xyz=0   0 rpy=0 0 0, axis 0 0 1, limit lower=-3.14159 upper=3.14159 effort=0.0 velocity=0.0
- added joint 440_413: type fixed, parent 440, child 413, origin xyz=0   0 rpy=0 0 0, axis 0 0 1, limit lower=-3.14159 upper=3.14159 effort=0.0 velocity=0.0
- added joint 440_414: type fixed, parent 440, child 414, origin xyz=0   0 rpy=0 0 0, axis 0 0 1, limit lower=-3.14159 upper=3.14159 effort=0.0 velocity=0.0
- added joint 440_415: type fixed, parent 440, child 415, origin xyz=0   0 rpy=0 0 0, axis 0 0 1, limit lower=-3.14159 upper=3.14159 effort=0.0 velocity=0.0
- added joint 440_416: type fixed, parent 440, child 416, origin xyz=0   0 rpy=0 0 0, axis 0 0 1, limit lower=-3.14159 upper=3.14159 effort=0.0 velocity=0.0
- added joint 440_421: type fixed, parent 440, child 421, origin xyz=0   0 rpy=0 0 0, axis 0 0 1, limit lower=-3.14159 upper=3.14159 effort=0.0 velocity=0.0
- added joint 440_431: type fixed, parent 440, child 431, origin xyz=0   0 rpy=0 0 0, axis 0 0 1, limit lower=-3.14159 upper=3.14159 effort=0.0 velocity=0.0
- added joint 440_441: type fixed, parent 440, child 441, origin xyz=0   0 rpy=0 0 0, axis 0 0 1, limit lower=-3.14159 upper=3.14159 effort=0.0 velocity=0.0
- added joint 440_451: type fixed, parent 440, child 451, origin xyz=0   0 rpy=0 0 0, axis 0 0 1, limit lower=-3.14159 upper=3.14159 effort=0.0 velocity=0.0
- added joint 440_461: type fixed, parent 440, child 461, origin xyz=0   0 rpy=0 0 0, axis 0 0 1, limit lower=-3.14159 upper=3.14159 effort=0.0 velocity=0.0
- added joint 440_472: type fixed, parent 440, child 472, origin xyz=0   0 rpy=0 0 0, axis 0 0 1, limit lower=-3.14159 upper=3.14159 effort=0.0 velocity=0.0
- added joint 440_473: type fixed, parent 440, child 473, origin xyz=0   0 rpy=0 0 0, axis 0 0 1, limit lower=-3.14159 upper=3.14159 effort=0.0 velocity=0.0
- added joint 440_474: type fixed, parent 440, child 474, origin xyz=0   0 rpy=0 0 0, axis 0 0 1, limit lower=-3.14159 upper=3.14159 effort=0.0 velocity=0.0
- added joint 440_475: type fixed, parent 440, child 475, origin xyz=0   0 rpy=0 0 0, axis 0 0 1, limit lower=-3.14159 upper=3.14159 effort=0.0 velocity=0.0
- added joint 440_476: type fixed, parent 440, child 476, origin xyz=0   0 rpy=0 0 0, axis 0 0 1, limit lower=-3.14159 upper=3.14159 effort=0.0 velocity=0.0
- added joint 440_512: type fixed, parent 440, child 512, origin xyz=0   0 rpy=0 0 0, axis 0 0 1, limit lower=-3.14159 upper=3.14159 effort=0.0 velocity=0.0
- added joint 440_513: type fixed, parent 440, child 513, origin xyz=0   0 rpy=0 0 0, axis 0 0 1, limit lower=-3.14159 upper=3.14159 effort=0.0 velocity=0.0
- added joint 440_514: type fixed, parent 440, child 514, origin xyz=0   0 rpy=0 0 0, axis 0 0 1, limit lower=-3.14159 upper=3.14159 effort=0.0 velocity=0.0
- added joint 440_515: type fixed, parent 440, child 515, origin xyz=0   0 rpy=0 0 0, axis 0 0 1, limit lower=-3.14159 upper=3.14159 effort=0.0 velocity=0.0
- added joint 440_516: type fixed, parent 440, child 516, origin xyz=0   0 rpy=0 0 0, axis 0 0 1, limit lower=-3.14159 upper=3.14159 effort=0.0 velocity=0.0
- added joint 440_521: type fixed, parent 440, child 521, origin xyz=0   0 rpy=0 0 0, axis 0 0 1, limit lower=-3.14159 upper=3.14159 effort=0.0 velocity=0.0
- added joint 440_531: type fixed, parent 440, child 531, origin xyz=0   0 rpy=0 0 0, axis 0 0 1, limit lower=-3.14159 upper=3.14159 effort=0.0 velocity=0.0
- added joint 440_541: type fixed, parent 440, child 541, origin xyz=0   0 rpy=0 0 0, axis 0 0 1, limit lower=-3.14159 upper=3.14159 effort=0.0 velocity=0.0
- added joint 440_551: type fixed, parent 440, child 551, origin xyz=0   0 rpy=0 0 0, axis 0 0 1, limit lower=-3.14159 upper=3.14159 effort=0.0 velocity=0.0
- added joint 440_561: type fixed, parent 440, child 561, origin xyz=0   0 rpy=0 0 0, axis 0 0 1, limit lower=-3.14159 upper=3.14159 effort=0.0 velocity=0.0
- added joint 440_572: type fixed, parent 440, child 572, origin xyz=0   0 rpy=0 0 0, axis 0 0 1, limit lower=-3.14159 upper=3.14159 effort=0.0 velocity=0.0
- added joint 440_573: type fixed, parent 440, child 573, origin xyz=0   0 rpy=0 0 0, axis 0 0 1, limit lower=-3.14159 upper=3.14159 effort=0.0 velocity=0.0
- added joint 440_574: type fixed, parent 440, child 574, origin xyz=0   0 rpy=0 0 0, axis 0 0 1, limit lower=-3.14159 upper=3.14159 effort=0.0 velocity=0.0
- added joint 440_575: type fixed, parent 440, child 575, origin xyz=0   0 rpy=0 0 0, axis 0 0 1, limit lower=-3.14159 upper=3.14159 effort=0.0 velocity=0.0
- added joint 440_576: type fixed, parent 440, child 576, origin xyz=0   0 rpy=0 0 0, axis 0 0 1, limit lower=-3.14159 upper=3.14159 effort=0.0 velocity=0.0
- added joint 440_613: type fixed, parent 440, child 613, origin xyz=0   0 rpy=0 0 0, axis 0 0 1, limit lower=-3.14159 upper=3.14159 effort=0.0 velocity=0.0
- added joint 440_614: type fixed, parent 440, child 614, origin xyz=0   0 rpy=0 0 0, axis 0 0 1, limit lower=-3.14159 upper=3.14159 effort=0.0 velocity=0.0
- added joint 440_615: type fixed, parent 440, child 615, origin xyz=0   0 rpy=0 0 0, axis 0 0 1, limit lower=-3.14159 upper=3.14159 effort=0.0 velocity=0.0
- added joint 440_622: type fixed, parent 440, child 622, origin xyz=0   0 rpy=0 0 0, axis 0 0 1, limit lower=-3.14159 upper=3.14159 effort=0.0 velocity=0.0
- added joint 440_626: type fixed, parent 440, child 626, origin xyz=0   0 rpy=0 0 0, axis 0 0 1, limit lower=-3.14159 upper=3.14159 effort=0.0 velocity=0.0
- added joint 440_631: type fixed, parent 440, child 631, origin xyz=0   0 rpy=0 0 0, axis 0 0 1, limit lower=-3.14159 upper=3.14159 effort=0.0 velocity=0.0
- added joint 440_641: type fixed, parent 440, child 641, origin xyz=0   0 rpy=0 0 0, axis 0 0 1, limit lower=-3.14159 upper=3.14159 effort=0.0 velocity=0.0
- added joint 440_651: type fixed, parent 440, child 651, origin xyz=0   0 rpy=0 0 0, axis 0 0 1, limit lower=-3.14159 upper=3.14159 effort=0.0 velocity=0.0
- added joint 440_662: type fixed, parent 440, child 662, origin xyz=0   0 rpy=0 0 0, axis 0 0 1, limit lower=-3.14159 upper=3.14159 effort=0.0 velocity=0.0
- added joint 440_666: type fixed, parent 440, child 666, origin xyz=0   0 rpy=0 0 0, axis 0 0 1, limit lower=-3.14159 upper=3.14159 effort=0.0 velocity=0.0
- added joint 440_673: type fixed, parent 440, child 673, origin xyz=0   0 rpy=0 0 0, axis 0 0 1, limit lower=-3.14159 upper=3.14159 effort=0.0 velocity=0.0
- added joint 440_674: type fixed, parent 440, child 674, origin xyz=0   0 rpy=0 0 0, axis 0 0 1, limit lower=-3.14159 upper=3.14159 effort=0.0 velocity=0.0
- added joint 440_675: type fixed, parent 440, child 675, origin xyz=0   0 rpy=0 0 0, axis 0 0 1, limit lower=-3.14159 upper=3.14159 effort=0.0 velocity=0.0
- added joint 440_723: type fixed, parent 440, child 723, origin xyz=0   0 rpy=0 0 0, axis 0 0 1, limit lower=-3.14159 upper=3.14159 effort=0.0 velocity=0.0
- added joint 440_724: type fixed, parent 440, child 724, origin xyz=0   0 rpy=0 0 0, axis 0 0 1, limit lower=-3.14159 upper=3.14159 effort=0.0 velocity=0.0
- added joint 440_725: type fixed, parent 440, child 725, origin xyz=0   0 rpy=0 0 0, axis 0 0 1, limit lower=-3.14159 upper=3.14159 effort=0.0 velocity=0.0
- added joint 440_732: type fixed, parent 440, child 732, origin xyz=0   0 rpy=0 0 0, axis 0 0 1, limit lower=-3.14159 upper=3.14159 effort=0.0 velocity=0.0
- added joint 440_733: type fixed, parent 440, child 733, origin xyz=0   0 rpy=0 0 0, axis 0 0 1, limit lower=-3.14159 upper=3.14159 effort=0.0 velocity=0.0
- added joint 440_734: type fixed, parent 440, child 734, origin xyz=0   0 rpy=0 0 0, axis 0 0 1, limit lower=-3.14159 upper=3.14159 effort=0.0 velocity=0.0
- added joint 440_735: type fixed, parent 440, child 735, origin xyz=0   0 rpy=0 0 0, axis 0 0 1, limit lower=-3.14159 upper=3.14159 effort=0.0 velocity=0.0
- added joint 440_736: type fixed, parent 440, child 736, origin xyz=0   0 rpy=0 0 0, axis 0 0 1, limit lower=-3.14159 upper=3.14159 effort=0.0 velocity=0.0
- added joint 440_742: type fixed, parent 440, child 742, origin xyz=0   0 rpy=0 0 0, axis 0 0 1, limit lower=-3.14159 upper=3.14159 effort=0.0 velocity=0.0
- added joint 440_743: type fixed, parent 440, child 743, origin xyz=0   0 rpy=0 0 0, axis 0 0 1, limit lower=-3.14159 upper=3.14159 effort=0.0 velocity=0.0
- added joint 440_744: type fixed, parent 440, child 744, origin xyz=0   0 rpy=0 0 0, axis 0 0 1, limit lower=-3.14159 upper=3.14159 effort=0.0 velocity=0.0
- added joint 440_745: type fixed, parent 440, child 745, origin xyz=0   0 rpy=0 0 0, axis 0 0 1, limit lower=-3.14159 upper=3.14159 effort=0.0 velocity=0.0
- added joint 440_746: type fixed, parent 440, child 746, origin xyz=0   0 rpy=0 0 0, axis 0 0 1, limit lower=-3.14159 upper=3.14159 effort=0.0 velocity=0.0
- added joint 440_752: type fixed, parent 440, child 752, origin xyz=0   0 rpy=0 0 0, axis 0 0 1, limit lower=-3.14159 upper=3.14159 effort=0.0 velocity=0.0
- added joint 440_753: type fixed, parent 440, child 753, origin xyz=0   0 rpy=0 0 0, axis 0 0 1, limit lower=-3.14159 upper=3.14159 effort=0.0 velocity=0.0
- added joint 440_754: type fixed, parent 440, child 754, origin xyz=0   0 rpy=0 0 0, axis 0 0 1, limit lower=-3.14159 upper=3.14159 effort=0.0 velocity=0.0
- added joint 440_755: type fixed, parent 440, child 755, origin xyz=0   0 rpy=0 0 0, axis 0 0 1, limit lower=-3.14159 upper=3.14159 effort=0.0 velocity=0.0
- added joint 440_756: type fixed, parent 440, child 756, origin xyz=0   0 rpy=0 0 0, axis 0 0 1, limit lower=-3.14159 upper=3.14159 effort=0.0 velocity=0.0
- added joint 440_763: type fixed, parent 440, child 763, origin xyz=0   0 rpy=0 0 0, axis 0 0 1, limit lower=-3.14159 upper=3.14159 effort=0.0 velocity=0.0
- added joint 440_764: type fixed, parent 440, child 764, origin xyz=0   0 rpy=0 0 0, axis 0 0 1, limit lower=-3.14159 upper=3.14159 effort=0.0 velocity=0.0
- added joint 440_765: type fixed, parent 440, child 765, origin xyz=0   0 rpy=0 0 0, axis 0 0 1, limit lower=-3.14159 upper=3.14159 effort=0.0 velocity=0.0
