Commit message: voxel cilia model

File: body84.urdf (robot description, URDF)
Before this commit: robot robot, 9 links, 8 joints
Links:
- removed link BackLeg
- removed link BackLower
- removed link FrontLeg
- removed link FrontLower
- removed link LeftLeg
- removed link LeftLower
- removed link RightLeg
- removed link RightLower
Joints:
- removed joint BackLeg_BackLower
- removed joint FrontLeg_FrontLower
- removed joint LeftLeg_LeftLower
- removed joint RightLeg_RightLower
- removed joint Torso_BackLeg
- removed joint Torso_FrontLeg
- removed joint Torso_LeftLeg
- removed joint Torso_RightLeg

File: body87.urdf (robot description, URDF)
Before this commit: robot robot, 9 links, 8 joints
Links:
- removed link BackLeg
- removed link BackLower
- removed link FrontLeg
- removed link FrontLower
- removed link LeftLeg
- removed link LeftLower
- removed link RightLeg
- removed link RightLower
Joints:
- removed joint BackLeg_BackLower
- removed joint FrontLeg_FrontLower
- removed joint LeftLeg_LeftLower
- removed joint RightLeg_RightLower
- removed joint Torso_BackLeg
- removed joint Torso_FrontLeg
- removed joint Torso_LeftLeg
- removed joint Torso_RightLeg
